Commit message: simple

File: LAB3/src/urdf/dynamicrobot.urdf (robot description, URDF)
Before this commit: robot kartezjan, 4 links, 3 joints
Links:
- link base_link: geometry visual cylinder length=3 radius=0.1
- link link1: geometry visual cylinder length=3 radius=0.1
- link link2: geometry visual cylinder length=3 radius=0.1
Joints:
- joint joint1: limit lower=0 upper=2 effort=30 velocity=1.0 -> lower=0 upper=3 effort=30 velocity=1.0; origin xyz=0 0 2 rpy=1.5708 1.5708 0  -> xyz=0 0 0 rpy=-1.5708 -1.5708 0 
- joint joint2: limit lower=0 upper=2 effort=30 velocity=1.0 -> lower=0 upper=3 effort=30 velocity=1.0; origin xyz=0 0 2 rpy=1.5708 1.5708 0  -> xyz=0 0 0 rpy=-1.5708 -1.5708 0 
- joint joint3: axis 0 0 -1 -> 0 0 1; limit lower=0 upper=2 effort=30 velocity=1.0 -> lower=0 upper=3 effort=30 velocity=1.0; origin xyz=0 0 2 rpy=0 0 0 -> xyz=0 0 0 rpy=0 0 0
