Commit message: co to ma byc

File: LAB4/src/urdf/dynamicrobot.urdf (robot description, URDF)
Before this commit: robot kartezjan, 4 links, 3 joints
Links:
- added link link0; visual box size=0.32 0.32 0.32
- link base_link: geometry visual box size=0.3 0.3 3.25
- link link1: geometry visual box size=0.25 0.25 3.2
- link link2: geometry visual box size=0.28 0.28 0.28
- link link3: geometry visual box size=0.2 0.2 3
Joints:
- added joint joint0: type fixed, parent link0, child link1
- joint joint1: child link1 -> link0
- joint joint2: limit lower=0 upper=3 effort=30 velocity=1.0 -> lower=0.3 upper=3 effort=30 velocity=1.0
- joint joint3: origin xyz=0 0 0 rpy=0 0 0 -> xyz=0 0 -3 rpy=0 0 0
